File: elec/layout/default/cafe-racer-taillight.kicad_pcb (KiCad board)
At the start: 2 copper layers, 225.7 x 100.8 mm, 0 parts

Commit message: initial design
Parts:
- added C1: 10.0 uF, lib:C0805, F.Cu at (233.4, 109.0)
- added C10: 100.0 nF, lib:C0402, F.Cu at (219.9, 122.6)
- added C11: 100.0 nF, lib:C0402, F.Cu at (219.9, 130.5)
- added C12: 1.0 uF, lib:C0402, F.Cu at (242.3, 125.4)
- added C13: 100.0 nF, lib:C0402, F.Cu at (237.4, 133.3)
- added C14: 100.0 nF, lib:C0402, F.Cu at (247.2, 133.3)
- added C15: 100.0 nF, lib:C0402, F.Cu at (226.2, 134.0)
- added C16: 1.0 uF, lib:C0402, F.Cu at (237.4, 129.4)
- added C17: 1.0 uF, lib:C0402, F.Cu at (219.9, 114.6)
- added C18: 1.0 uF, lib:C0402, F.Cu at (247.2, 129.4)
- added C2: 10.0 uF, lib:C0805, F.Cu at (239.9, 109.0)
- added C3: 10.0 uF, lib:C0805, F.Cu at (227.0, 109.0)
- added C4: 100.0 nF, lib:C0402, F.Cu at (237.4, 125.4)
- added C5: 22.0 pF, lib:C0402, F.Cu at (242.3, 129.4)
- added C6: 22.0 pF, lib:C0402, F.Cu at (219.9, 118.6)
- added C7: 100.0 nF, lib:C0402, F.Cu at (247.2, 125.4)
- added C8: 100.0 nF, lib:C0402, F.Cu at (219.9, 126.5)
- added C9: 100.0 nF, lib:C0402, F.Cu at (242.3, 133.3)
- added R1: 51.0 KΩ, lib:R0402, F.Cu at (232.5, 125.4)
- added R10: 10.0 KΩ, lib:R0402, F.Cu at (232.5, 133.4)
- added R11: 10.0 KΩ, lib:R0402, F.Cu at (242.4, 117.4)
- added R12: 10.0 KΩ, lib:R0402, F.Cu at (247.3, 113.5)
- added R13: 10.0 KΩ, lib:R0402, F.Cu at (247.3, 121.4)
- added R14: 10.0 KΩ, lib:R0402, F.Cu at (247.3, 117.4)
- added R15: 10.0 KΩ, lib:R0402, F.Cu at (242.4, 121.4)
- added R16: 10.0 KΩ, lib:R0402, F.Cu at (232.5, 117.4)
- added R17: 10.0 KΩ, lib:R0402, F.Cu at (232.5, 129.4)
- added R18: 5.1 KΩ, lib:R0402, F.Cu at (232.5, 113.5)
- added R19: 5.1 KΩ, lib:R0402, F.Cu at (232.5, 121.4)
- added R2: 10.0 KΩ, lib:R0402, F.Cu at (226.2, 122.0)
- added R3: 1.0 KΩ, lib:R0402, F.Cu at (237.4, 113.5)
- added R4: 27.0 KΩ, lib:R0402, F.Cu at (237.4, 121.4)
- added R5: 27.0 KΩ, lib:R0402, F.Cu at (226.2, 126.0)
- added R6: 10.0 KΩ, lib:R0402, F.Cu at (242.4, 113.5)
- added R7: 10.0 KΩ, lib:R0402, F.Cu at (237.4, 117.4)
- added R8: 18.0 KΩ, lib:R0402, F.Cu at (226.2, 130.0)
- added R9: 10.0 KΩ, lib:R0402, F.Cu at (226.2, 118.1)
- added U1: , lib:SOT-23-6_L2.9-W1.6-P0.95-LS2.8-BR, F.Cu at (227.2, 103.8)
- added U10: , lib:SOT-23-3_L2.9-W1.3-P1.90-LS2.4-BR, F.Cu at (247.4, 102.8)
- added U11: , lib:SOT-23-3_L2.9-W1.3-P1.90-LS2.4-BR, F.Cu at (206.7, 104.1)
- added U12: , lib:USB-C-SMD_KH-TYPE-C-16P, F.Cu at (171.4, 123.2)
- added U13: , lib:CONN-TH_5P-P5.00_WJ127-5.0-5P, F.Cu at (206.9, 83.8)
- added U14: , lib:CONN-TH_3P-P5.00_WJ127-5.0-3P, F.Cu at (204.5, 139.7)
- added U2: , lib:SOD-323_L1.8-W1.3-LS2.5-RD, F.Cu at (226.9, 113.8)
- added U3: , lib:L0805, F.Cu at (246.4, 108.8)
- added U4: , lib:LQFN-56_L7.0-W7.0-P0.4-EP, F.Cu at (195.1, 106.4)
- added U5: , lib:OSC-SMD_4P-L3.2-W2.5-BL, F.Cu at (194.1, 113.9)
- added U6: , lib:SOIC-8_L5.3-W5.3-P1.27-LS8.0-BL, F.Cu at (192.1, 97.2)
- added U8: , lib:SOT-23-3_L2.9-W1.3-P1.90-LS2.4-BR, F.Cu at (241.1, 102.8)
- added U9: , lib:SOT-23-3_L2.9-W1.3-P1.90-LS2.4-BR, F.Cu at (234.9, 102.8)
